File: MicroMousePower.kicad_pcb (KiCad board)
At the start: 2 copper layers, 59.6 x 56 mm, 105 parts, among them J1 USB_C_Receptacle_PowerOnly_6P, J2 Conn_02x16_Odd_Even, J3 Conn_01x02_Pin, Q1 TIP41C, Q2 TIP41C, Q3 TIP41C, U1 INA219AxDCN, U2 MCP73831-3-MC, U3 CH224K, U4 DRV8833PWPR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

Commit message: the pain never ends
Parts:
- moved U7 23.4 mm to (190.3, 108.7), turned to -90 degrees
- moved C2 4.11 mm to (191.0, 99.5)
- moved U6 4.11 mm to (191.1, 97.4)
- moved R26 4.06 mm to (191.0, 104.5)
- moved C9 4.01 mm to (191.0, 85.8)
- moved R14 4.01 mm to (190.9, 89.5)
- moved R15 4.01 mm to (191.1, 93.0)
- moved C13 1.83 mm to (162.1, 93.5)
- moved R7 1.10 mm to (168.5, 84.5)
- moved R22 0.80 mm to (161.6, 89.0)
- moved U9 0.30 mm to (168.5, 91.5)
- renumbered C2 to C52
Routing:
- net -BATT: track 0.00 -> 341.8 mm, vias 0 -> 10
- net +BATT: track 0.00 -> 268.5 mm, vias 0 -> 7
- net /3V3: track 0.00 -> 195.1 mm, vias 0 -> 4
- net /5V: track 0.00 -> 176.1 mm, vias 0 -> 5
- net /USB 5V: track 0.00 -> 104.9 mm, vias 0 -> 6
- net /9V: track 0.00 -> 86.2 mm, vias 0 -> 4
- net /EXT_LOAD1_OUT: track 0.00 -> 82.6 mm, vias 0 -> 3
- net /EXT_LOAD2_OUT: track 0.00 -> 78.5 mm, vias 0 -> 2
- net Net-(D1-PadC): track 0.00 -> 67.0 mm, vias 0 -> 3
- net Net-(D2-PadC): track 0.00 -> 63.7 mm, vias 0 -> 3
- net Net-(U7-SW): track 0.00 -> 61.0 mm, vias 0 -> 3
- net Net-(U8-EN): track 0.00 -> 49.2 mm
- net Net-(U1-IN-): track 0.00 -> 48.8 mm
- net /I2C1_SCL: track 0.00 -> 48.3 mm, vias 0 -> 2
- net Net-(R2-Pad1): track 0.00 -> 45.6 mm, vias 0 -> 2
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Other:
- board size 59.6 x 56 mm -> 58.6 x 55 mm
