File: MicroMousePower.kicad_pcb (KiCad board)
At the start: 2 copper layers, 58.6 x 55 mm, 104 parts, among them J1 USB_C_Receptacle_PowerOnly_6P, J2 Conn_02x16_Odd_Even, J3 Conn_01x02_Pin, Q1 TIP41C, Q2 TIP41C, Q3 TIP41C, U1 INA219AxDCN, U2 MCP73831-3-MC, U3 CH224K, U4 DRV8833PWPR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

Commit message: final submission
Parts:
- added R45: 10, Resistor_SMD:R_1206_3216Metric, F.Cu at (190.0, 107.0)
- added R46: 10, Resistor_SMD:R_1206_3216Metric, F.Cu at (190.0, 111.0)
- added R47: 10, Resistor_SMD:R_1206_3216Metric, F.Cu at (171.5, 75.0)
- added R48: 10, Resistor_SMD:R_1206_3216Metric, F.Cu at (175.5, 74.5)
- moved R27 7.91 mm to (179.5, 77.5)
- moved U1 2.46 mm to (179.0, 74.5)
Connections:
- C52 pad 1: /3V3 -> Net-(U9-VO)
- U9 pad 3: /3V3 -> Net-(U9-VO)
Routing:
- net -BATT: track 0.00 -> 317.8 mm, vias 0 -> 9
- net +BATT: track 0.00 -> 271.4 mm, vias 0 -> 7
- net /3V3: track 0.00 -> 172.6 mm, vias 0 -> 6
- net /5V: track 0.00 -> 166.6 mm, vias 0 -> 6
- net /USB 5V: track 0.00 -> 101.5 mm, vias 0 -> 3
- net /9V: track 0.00 -> 84.5 mm, vias 0 -> 5
- net /EXT_LOAD2_OUT: track 0.00 -> 83.0 mm, vias 0 -> 3
- net /EXT_LOAD1_OUT: track 0.00 -> 77.6 mm, vias 0 -> 2
- net /I2C1_SDA: track 0.00 -> 68.4 mm, vias 0 -> 3
- net Net-(R45-Pad2): track 0.00 -> 66.8 mm, vias 0 -> 2
- net Net-(D1-PadC): track 0.00 -> 62.1 mm, vias 0 -> 3
- net Net-(D2-PadC): track 0.00 -> 56.8 mm, vias 0 -> 3
- net Net-(Q2-B): track 0.00 -> 54.0 mm, vias 0 -> 3
- net Net-(U8-EN): track 0.00 -> 52.4 mm, vias 0 -> 3
- net Net-(R2-Pad1): track 0.00 -> 45.5 mm, vias 0 -> 3
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Other:
- board text added: "push these buttons to kaboom"
